File: backup/LeftSensor.sch (EAGLE design)
At the start: 9 parts, among them X2 CNY70

Commit message: Added code V1
Parts:
- removed PAD4, PAD5, PAD6: WIREPADSMD1,27-254, wirepad:WIREPADSMD1,27-254
- removed X1: (no value), tom:USB-MB-S
Connections:
- removed net SENSOR1: PAD2.P, X1.VBUS
- removed net SENSOR2: X1.D-, X2.EMI
- removed net SENSOR3: PAD5.P, X1.ID
- new net SENSOR: PAD2.P, X2.EMI
- net GND: no longer PAD6.P, X1.GND
- net VCC: no longer PAD4.P, X1.D+
Other:
- moved on the sheet: PAD1, PAD2, PAD3, R1, X2
Changed lines of the file:
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@@
 <settings>
 <setting alwaysvectorfont="no"/>
-<setting keepoldvectorfont="yes"/>
 <setting verticaltext="up"/>
 </settings>
@@
 <layer number="88" name="SimResults" color="9" fill="1" visible="yes" active="yes"/>
 <layer number="89" name="SimProbes" color="9" fill="1" visible="yes" active="yes"/>
-<layer number="90" name="Modules" color="5" fill="1" visible="no" active="yes"/>
+<layer number="90" name="Modules" color="5" fill="1" visible="yes" active="yes"/>
 <layer number="91" name="Nets" color="2" fill="1" visible="yes" active="yes"/>
 <layer number="92" name="Busses" color="1" fill="1" visible="yes" active="yes"/>
@@
 <parts>
 <part name="R1" library="ScyllAlarmV3.0" deviceset="RCL_R-EU_" device="R0805"/>
-<part name="X1" library="tom" deviceset="USB" device="-MB-S"/>
 <part name="X2" library="cny70" deviceset="CNY70" device=""/>
 <part name="PAD1" library="wirepad" library_urn="urn:adsk.eagle:library:412" deviceset="WIREPAD" device="SMD1,27-254" package3d_urn="urn:adsk.eagle:package:30839/1" value="WIREPADSMD1,27-254"/>
 <part name="PAD2" library="wirepad" deviceset="WIREPAD" device="SMD1,27-254" value="WIREPADSMD1,27-254"/>
 <part name="PAD3" library="wirepad" deviceset="WIREPAD" device="SMD1,27-254" value="WIREPADSMD1,27-254"/>
-<part name="PAD4" library="wirepad" deviceset="WIREPAD" device="SMD1,27-254" value="WIREPADSMD1,27-254"/>
-<part name="PAD5" library="wirepad" deviceset="WIREPAD" device="SMD1,27-254" value="WIREPADSMD1,27-254"/>
-<part name="PAD6" library="wirepad" deviceset="WIREPAD" device="SMD1,27-254" value="WIREPADSMD1,27-254"/>
 </parts>
 <sheets>
@@
 </plain>
 <instances>
-<instance part="R1" gate="G$1" x="38.1" y="60.96"/>
-<instance part="X1" gate="G$1" x="88.9" y="78.74"/>
-<instance part="X2" gate="G$1" x="55.88" y="63.5"/>
-<instance part="PAD1" gate="G$1" x="25.4" y="90.17" smashed="yes">
-<attribute name="NAME" x="24.257" y="92.0242" size="1.778" layer="95"/>
+<instance part="R1" gate="G$1" x="45.72" y="30.48"/>
+<instance part="X2" gate="G$1" x="63.5" y="33.02"/>
+<instance part="PAD1" gate="G$1" x="33.02" y="59.69" smashed="yes">
+<attribute name="NAME" x="31.877" y="61.5442" size="1.778" layer="95"/>
 </instance>
-<instance part="PAD2" gate="G$1" x="25.4" y="83.82" smashed="yes">
-<attribute name="NAME" x="24.257" y="85.6742" size="1.778" layer="95"/>
+<instance part="PAD2" gate="G$1" x="33.02" y="53.34" smashed="yes">
+<attribute name="NAME" x="31.877" y="55.1942" size="1.778" layer="95"/>
 </instance>
-<instance part="PAD3" gate="G$1" x="25.4" y="77.47" smashed="yes">
-<attribute name="NAME" x="24.257" y="79.3242" size="1.778" layer="95"/>
-</instance>
-<instance part="PAD4" gate="G$1" x="45.72" y="90.17" smashed="yes">
-<attribute name="NAME" x="44.577" y="92.0242" size="1.778" layer="95"/>
-</instance>
-<instance part="PAD5" gate="G$1" x="45.72" y="83.82" smashed="yes">
-<attribute name="NAME" x="44.577" y="85.6742" size="1.778" layer="95"/>
-</instance>
-<instance part="PAD6" gate="G$1" x="45.72" y="77.47" smashed="yes">
-<attribute name="NAME" x="44.577" y="79.3242" size="1.778" layer="95"/>
+<instance part="PAD3" gate="G$1" x="33.02" y="46.99" smashed="yes">
+<attribute name="NAME" x="31.877" y="48.8442" size="1.778" layer="95"/>
 </instance>
 </instances>
@@
 </busses>
 <nets>
-<net name="SENSOR1" class="0">
+<net name="SENSOR" class="0">
 <segment>
 <pinref part="PAD2" gate="G$1" pin="P"/>
-<wire x1="27.94" y1="83.82" x2="38.1" y2="83.82" width="0.1524" layer="91"/>
-<label x="30.48" y="83.82" size="1.778" layer="95"/>
-</segment>
-<segment>
-<pinref part="X1" gate="G$1" pin="VBUS"/>
-<wire x1="86.36" y1="82.55" x2="73.66" y2="82.55" width="0.1524" layer="91"/>
-<label x="69.85" y="82.55" size="1.778" layer="95"/>
+<wire x1="35.56" y1="53.34" x2="45.72" y2="53.34" width="0.1524" layer="91"/>
+<label x="38.1" y="53.34" size="1.778" layer="95"/>
+</segment>
+<segment>
+<pinref part="X2" gate="G$1" pin="EMI"/>
+<wire x1="71.12" y1="30.48" x2="77.47" y2="30.48" width="0.1524" layer="91"/>
+<label x="72.39" y="30.48" size="1.778" layer="95"/>
 </segment>
 </net>
 <net name="SENSOR2" class="0">
 <segment>
-<pinref part="X2" gate="G$1" pin="EMI"/>
-<wire x1="63.5" y1="60.96" x2="69.85" y2="60.96" width="0.1524" layer="91"/>
-<label x="64.77" y="60.96" size="1.778" layer="95"/>
-</segment>
-<segment>
-<pinref part="X1" gate="G$1" pin="D-"/>
-<wire x1="86.36" y1="85.09" x2="73.66" y2="85.09" width="0.1524" layer="91"/>
-<label x="69.85" y="85.09" size="1.778" layer="95"/>
-</segment>
-</net>
-<net name="SENSOR3" class="0">
-<segment>
-<pinref part="X1" gate="G$1" pin="ID"/>
-<wire x1="86.36" y1="77.47" x2="73.66" y2="77.47" width="0.1524" layer="91"/>
-<label x="69.85" y="77.47" size="1.778" layer="95"/>
-</segment>
-<segment>
-<pinref part="PAD5" gate="G$1" pin="P"/>
-<wire x1="48.26" y1="83.82" x2="58.42" y2="83.82" width="0.1524" layer="91"/>
-<label x="50.8" y="83.82" size="1.778" layer="95"/>
+<wire x1="93.98" y1="54.61" x2="81.28" y2="54.61" width="0.1524" layer="91"/>
 </segment>
 </net>
@@
 <segment>
 <pinref part="X2" gate="G$1" pin="A"/>
-<wire x1="45.72" y1="66.04" x2="38.1" y2="66.04" width="0.1524" layer="91"/>
-<label x="38.1" y="66.04" size="1.778" layer="95"/>
+<wire x1="53.34" y1="35.56" x2="45.72" y2="35.56" width="0.1524" layer="91"/>
+<label x="45.72" y="35.56" size="1.778" layer="95"/>
 </segment>
 <segment>
 <pinref part="X2" gate="G$1" pin="COL"/>
-<wire x1="63.5" y1="66.04" x2="69.85" y2="66.04" width="0.1524" layer="91"/>
-<label x="64.77" y="66.04" size="1.778" layer="95"/>
+<wire x1="71.12" y1="35.56" x2="77.47" y2="35.56" width="0.1524" layer="91"/>
+<label x="72.39" y="35.56" size="1.778" layer="95"/>
 </segment>
 <segment>
 <pinref part="PAD1" gate="G$1" pin="P"/>
-<wire x1="27.94" y1="90.17" x2="38.1" y2="90.17" width="0.1524" layer="91"/>
-<label x="33.02" y="91.44" size="1.778" layer="95"/>
-</segment>
-<segment>
-<pinref part="PAD4" gate="G$1" pin="P"/>
-<wire x1="48.26" y1="90.17" x2="58.42" y2="90.17" width="0.1524" layer="91"/>
-<label x="53.34" y="91.44" size="1.778" layer="95"/>
-</segment>
-<segment>
-<pinref part="X1" gate="G$1" pin="D+"/>
-<wire x1="86.36" y1="87.63" x2="73.66" y2="87.63" width="0.1524" layer="91"/>
-<label x="69.85" y="87.63" size="1.778" layer="95"/>
+<wire x1="35.56" y1="59.69" x2="45.72" y2="59.69" width="0.1524" layer="91"/>
+<label x="40.64" y="60.96" size="1.778" layer="95"/>
 </segment>
 </net>
 <net name="GND" class="0">
 <segment>
-<pinref part="X1" gate="G$1" pin="GND"/>
-<wire x1="86.36" y1="80.01" x2="73.66" y2="80.01" width="0.1524" layer="91"/>
-<label x="69.85" y="80.01" size="1.778" layer="95"/>
-</segment>
-<segment>
 <pinref part="R1" gate="G$1" pin="1"/>
-<wire x1="33.02" y1="60.96" x2="27.94" y2="60.96" width="0.1524" layer="91"/>
-<label x="27.94" y="60.96" size="1.778" layer="95"/>
+<wire x1="40.64" y1="30.48" x2="35.56" y2="30.48" width="0.1524" layer="91"/>
+<label x="35.56" y="30.48" size="1.778" layer="95"/>
 </segment>
 <segment>
 <pinref part="PAD3" gate="G$1" pin="P"/>
-<wire x1="27.94" y1="77.47" x2="38.1" y2="77.47" width="0.1524" layer="91"/>
-<label x="33.02" y="78.74" size="1.778" layer="95"/>
-</segment>
-<segment>
-<pinref part="PAD6" gate="G$1" pin="P"/>
-<wire x1="48.26" y1="77.47" x2="58.42" y2="77.47" width="0.1524" layer="91"/>
-<label x="53.34" y="78.74" size="1.778" layer="95"/>
+<wire x1="35.56" y1="46.99" x2="45.72" y2="46.99" width="0.1524" layer="91"/>
+<label x="40.64" y="48.26" size="1.778" layer="95"/>
 </segment>
 </net>
@@
 <pinref part="R1" gate="G$1" pin="2"/>
 <pinref part="X2" gate="G$1" pin="C"/>
-<wire x1="43.18" y1="60.96" x2="45.72" y2="60.96" width="0.1524" layer="91"/>
-</segment>
-</net>
+<wire x1="50.8" y1="30.48" x2="53.34" y2="30.48" width="0.1524" layer="91"/>
+</segment>
+</net>
